Commit message: Checkpoint physical target simulation and validation WIP

File: resources/models/environment_assets/objects/navrl_target_drone.urdf (robot description, URDF)
Before this commit: robot navrl_target_drone, 1 links, 0 joints
Links:
- link base_link: mass 0.25 -> 1.20; geometry collision box size=0.28 0.28 0.12; visual box size=0.28 0.28 0.12
