Commit message: Measure the new target in the real simulator: it never reaches the detector
V1 was verified only in the isolated renderer. Running it through Isaac Gym and
the detector's own camera found two things, neither expected.

The asset did not load at all. warp_asset.py indexes a per-link name list with a
per-mesh counter, so it assumes one mesh per link, and thirteen visuals in one
link raised IndexError before a frame was drawn. Rather than change shared
simulator code, the asset now has the shape the interceptor URDF already uses:
one visual per link, fixed joints, added links massless and without collision,
base_link's inertial and collision untouched. It loads.

Once loading, the detector sees exactly the same thing either way. Across 3,840
paired samples at 32 environments, with identical trajectories because
appearance does not affect physics, the area ratio is 1.000 with an
interquartile range of 1.000 to 1.000, in every range bin.

The reason is in the mask kernel: it intersects rays with an analytic sphere or
an oriented box whose half extents are hard-coded, and uses the mesh only to
test occlusion by bars. The target's visual geometry is not in that path, so no
change to the URDF can move what the detector sees.

That reorders the plan. Making the target look like a drone needs the detector's
target rendering changed from an analytic proxy to real geometry, and that comes
before the shading work, not after. The prototype's 41% area drop describes a
renderer the pipeline does not use; the confound it implies starts to apply only
once the detector reads meshes.

Two runs returned zero pixels everywhere first. Zero actions never pointed the
camera at the target, and after fixing that the probe was reading
last_pixel_count, which is the detection path's post-gating count and stayed 0
while target_mask held 48 to 55 pixels. Taking a plausible-looking field name
without checking it is what cost those runs.

Co-Authored-By: Claude Opus 5 (1M context) <noreply@anthropic.com>

File: resources/models/environment_assets/objects/navrl_target_drone_v3.urdf (robot description, URDF)
Before this commit: robot navrl_target_drone_v3, 1 links, 0 joints
Links:
- added link arm_0, mass 0.0; visual cylinder length=0.11 radius=0.01
- added link arm_1, mass 0.0; visual cylinder length=0.11 radius=0.01
- added link arm_2, mass 0.0; visual cylinder length=0.11 radius=0.01
- added link arm_3, mass 0.0; visual cylinder length=0.11 radius=0.01
- added link motor_0, mass 0.0; visual cylinder length=0.05 radius=0.01
- added link motor_1, mass 0.0; visual cylinder length=0.05 radius=0.01
- added link motor_2, mass 0.0; visual cylinder length=0.05 radius=0.01
- added link motor_3, mass 0.0; visual cylinder length=0.05 radius=0.01
- added link prop_0, mass 0.0; visual cylinder length=0.006 radius=0.0635
- added link prop_1, mass 0.0; visual cylinder length=0.006 radius=0.0635
- added link prop_2, mass 0.0; visual cylinder length=0.006 radius=0.0635
- added link prop_3, mass 0.0; visual cylinder length=0.006 radius=0.0635
- link base_link: geometry collision box size=0.283 0.283 0.12; visual box size=0.15 0.15 0.12
Joints:
- added joint base_link_to_arm_0: type fixed, parent base_link, child arm_0, origin xyz=0.03889085 -0.03889085 0.0 rpy=0.0 1.5707963267948966 -0.7853981633974483
- added joint base_link_to_arm_1: type fixed, parent base_link, child arm_1, origin xyz=-0.03889085 -0.03889085 0.0 rpy=0.0 1.5707963267948966 -2.356194490192345
- added joint base_link_to_arm_2: type fixed, parent base_link, child arm_2, origin xyz=-0.03889085 0.03889085 0.0 rpy=0.0 1.5707963267948966 2.356194490192345
- added joint base_link_to_arm_3: type fixed, parent base_link, child arm_3, origin xyz=0.03889085 0.03889085 0.0 rpy=0.0 1.5707963267948966 0.7853981633974483
- added joint base_link_to_motor_0: type fixed, parent base_link, child motor_0, origin xyz=0.0777817 -0.0777817 0.0 rpy=0.0 0.0 0.0
- added joint base_link_to_motor_1: type fixed, parent base_link, child motor_1, origin xyz=-0.0777817 -0.0777817 0.0 rpy=0.0 0.0 0.0
- added joint base_link_to_motor_2: type fixed, parent base_link, child motor_2, origin xyz=-0.0777817 0.0777817 0.0 rpy=0.0 0.0 0.0
- added joint base_link_to_motor_3: type fixed, parent base_link, child motor_3, origin xyz=0.0777817 0.0777817 0.0 rpy=0.0 0.0 0.0
- added joint base_link_to_prop_0: type fixed, parent base_link, child prop_0, origin xyz=0.0777817 -0.0777817 0.028 rpy=0.0 0.0 0.0
- added joint base_link_to_prop_1: type fixed, parent base_link, child prop_1, origin xyz=-0.0777817 -0.0777817 0.028 rpy=0.0 0.0 0.0
- added joint base_link_to_prop_2: type fixed, parent base_link, child prop_2, origin xyz=-0.0777817 0.0777817 0.028 rpy=0.0 0.0 0.0
- added joint base_link_to_prop_3: type fixed, parent base_link, child prop_3, origin xyz=0.0777817 0.0777817 0.028 rpy=0.0 0.0 0.0
